Commit message: 里程计完美标定+SLAM建图完成: wheel_radius=0.06475, wheel_separation=0.23364, 闭环精度0.072%(2.31cm), 工业AGV级别

File: src/robot_bringup_cpp/urdf/my_robot.urdf.xacro (robot description, xacro)
@@ -25,5 +25,5 @@
       <origin rpy="1.5707 0 0" xyz="0 0 0"/>
       <geometry>
-        <cylinder length="0.051" radius="0.064"/>
+        <cylinder length="0.051" radius="0.06475"/>
       </geometry>
       <material name="grey_material">
@@ -34,5 +34,5 @@
       <origin rpy="1.5707 0 0" xyz="0 0 0"/>
       <geometry>
-        <cylinder length="0.051" radius="0.064"/>
+        <cylinder length="0.051" radius="0.06475"/>
       </geometry>
     </collision>
@@ -46,5 +46,5 @@
       <origin rpy="1.5707 0 0" xyz="0 0 0"/>
       <geometry>
-        <cylinder length="0.051" radius="0.064"/>
+        <cylinder length="0.051" radius="0.06475"/>
       </geometry>
       <material name="grey_material">
@@ -55,5 +55,5 @@
       <origin rpy="1.5707 0 0" xyz="0 0 0"/>
       <geometry>
-        <cylinder length="0.051" radius="0.064"/>
+        <cylinder length="0.051" radius="0.06475"/>
       </geometry>
     </collision>
@@ -66,10 +66,10 @@
     <parent link="base_footprint"/>
     <child link="base_link"/>
-    <origin xyz="0 0 0.222" rpy="0 0 0"/>  <!-- 修正: 0.222 + (-0.158) = 0.064 (轮半径) -->
+    <origin xyz="0 0 0.222" rpy="0 0 0"/>  <!-- 修正: 0.222 + (-0.158) = 0.06475 (轮半径-直线标定11cm) -->
   </joint>
   <joint name="left_wheel_joint" type="continuous">
     <parent link="base_link"/>
     <child link="left_wheel_link"/>
-    <origin rpy="0 0 0" xyz="0 0.114 -0.158"/>  <!-- 轮距22.8cm/2=11.4cm（360°标定修正：348.4°→360°）, 轮心离地6.4cm -->
+    <origin rpy="0 0 0" xyz="0 0.11682 -0.158"/>  <!-- 轮距23.364cm/2=11.682cm（线性插值：2圈少转10.5°，3圈多转6.1°）, 轮心离地6.4cm -->
     <axis xyz="0 1 0"/>
   </joint>
@@ -77,5 +77,5 @@
     <parent link="base_link"/>
     <child link="right_wheel_link"/>
-    <origin rpy="0 0 0" xyz="0 -0.114 -0.158"/>  <!-- 轮距22.8cm/2=11.4cm（360°标定修正：348.4°→360°）, 轮心离地6.4cm -->
+    <origin rpy="0 0 0" xyz="0 -0.11682 -0.158"/>  <!-- 轮距23.364cm/2=11.682cm（线性插值：2圈少转10.5°，3圈多转6.1°）, 轮心离地6.4cm -->
     <axis xyz="0 1 0"/>
   </joint>

Commit message: 标定更新: USB端口映射修复 + 轮径/轮距参数调整
- 修复USB端口映射: serial_bridge(USB0), imu_publisher(USB1), odom_publisher(USB2)
- 轮径标定: 0.0645m
- 轮距标定: 0.23364m
- 更新所有相关文件: C++节点、launch文件、URDF

File: src/robot_bringup_cpp/urdf/my_robot.urdf.xacro (robot description, xacro)
@@ -25,5 +25,5 @@
       <origin rpy="1.5707 0 0" xyz="0 0 0"/>
       <geometry>
-        <cylinder length="0.051" radius="0.06475"/>
+        <cylinder length="0.051" radius="0.0645"/>
       </geometry>
       <material name="grey_material">
@@ -34,5 +34,5 @@
       <origin rpy="1.5707 0 0" xyz="0 0 0"/>
       <geometry>
-        <cylinder length="0.051" radius="0.06475"/>
+        <cylinder length="0.051" radius="0.0645"/>
       </geometry>
     </collision>
@@ -46,5 +46,5 @@
       <origin rpy="1.5707 0 0" xyz="0 0 0"/>
       <geometry>
-        <cylinder length="0.051" radius="0.06475"/>
+        <cylinder length="0.051" radius="0.0645"/>
       </geometry>
       <material name="grey_material">
@@ -55,5 +55,5 @@
       <origin rpy="1.5707 0 0" xyz="0 0 0"/>
       <geometry>
-        <cylinder length="0.051" radius="0.06475"/>
+        <cylinder length="0.051" radius="0.0645"/>
       </geometry>
     </collision>
@@ -66,5 +66,5 @@
     <parent link="base_footprint"/>
     <child link="base_link"/>
-    <origin xyz="0 0 0.222" rpy="0 0 0"/>  <!-- 修正: 0.222 + (-0.158) = 0.06475 (轮半径-直线标定11cm) -->
+    <origin xyz="0 0 0.2225" rpy="0 0 0"/>  <!-- 修正: 0.2225 + (-0.158) = 0.0645 (轮半径-标定值0.0645m) -->
   </joint>
   <joint name="left_wheel_joint" type="continuous">

Commit message: 更新导航系统：保存高精度地图(0.8cm)到src/map2，优化导航参数配置

File: src/robot_bringup_cpp/urdf/my_robot.urdf.xacro (robot description, xacro)
@@ -5,5 +5,5 @@
     <visual>
       <geometry>
-        <box size="0.45 0.38 0.15" />
+        <box size="0.45 0.38 0.5" />
       </geometry>
       <material name="blue_material">
@@ -13,5 +13,5 @@
     <collision>
       <geometry>
-        <box size="0.45 0.38 0.15" />
+        <box size="0.45 0.38 0.5" />
       </geometry>
     </collision>
@@ -66,10 +66,35 @@
     <parent link="base_footprint"/>
     <child link="base_link"/>
-    <origin xyz="0 0 0.2225" rpy="0 0 0"/>  <!-- 修正: 0.2225 + (-0.158) = 0.0645 (轮半径-标定值0.0645m) -->
+    <origin xyz="0 0 0.398" rpy="0 0 0"/>  <!-- 2025-11-15更新: 底盘高50cm，中心离地39.8cm（轮心6.45cm + 底盘下沿到中心25cm） -->
+  </joint>
+  <!-- 新增：中心立柱结构 14.4cm×14.4cm×100cm -->
+  <link name="center_pillar_link">
+    <visual>
+      <geometry>
+        <box size="0.144 0.144 1.0" />
+      </geometry>
+      <material name="pillar_material">
+        <color rgba="0.3 0.3 0.3 0.9" />  <!-- 深灰色 -->
+      </material>
+    </visual>
+    <collision>
+      <geometry>
+        <box size="0.144 0.144 1.0" />
+      </geometry>
+    </collision>
+    <inertial>
+      <mass value="5.0" />
+      <inertia ixx="0.42" ixy="0.0" ixz="0.0" iyy="0.42" iyz="0.0" izz="0.01" />
+    </inertial>
+  </link>
+  <joint name="center_pillar_joint" type="fixed">
+    <parent link="base_link"/>
+    <child link="center_pillar_link"/>
+    <origin xyz="0 0 0.25" rpy="0 0 0"/>  <!-- 立柱中心相对base_link向上25cm，使立柱底面与底盘底面重合 -->
   </joint>
   <joint name="left_wheel_joint" type="continuous">
     <parent link="base_link"/>
     <child link="left_wheel_link"/>
-    <origin rpy="0 0 0" xyz="0 0.11682 -0.158"/>  <!-- 轮距23.364cm/2=11.682cm（线性插值：2圈少转10.5°，3圈多转6.1°）, 轮心离地6.4cm -->
+    <origin rpy="0 0 0" xyz="0 0.11682 -0.3335"/>  <!-- 2025-11-15更新: 轮距23.364cm/2=11.682cm, 底盘高50cm后轮心相对base_link为-33.35cm -->
     <axis xyz="0 1 0"/>
   </joint>
@@ -77,5 +102,5 @@
     <parent link="base_link"/>
     <child link="right_wheel_link"/>
-    <origin rpy="0 0 0" xyz="0 -0.11682 -0.158"/>  <!-- 轮距23.364cm/2=11.682cm（线性插值：2圈少转10.5°，3圈多转6.1°）, 轮心离地6.4cm -->
+    <origin rpy="0 0 0" xyz="0 -0.11682 -0.3335"/>  <!-- 2025-11-15更新: 轮距23.364cm/2=11.682cm, 底盘高50cm后轮心相对base_link为-33.35cm -->
     <axis xyz="0 1 0"/>
   </joint>
@@ -102,5 +127,5 @@
     <parent link="base_link"/>
     <child link="laser_link"/>
-    <origin xyz="0.157 0 0.214" rpy="0 0 0"/>  <!-- 修正+0.002: 思岚S2L精确实测 -->
+    <origin xyz="0.258 0 0.318" rpy="0 0 0"/>  <!-- 2025-11-15更新: 底盘高50cm，雷达底部仍离地69.6cm，雷达中心相对base_link为31.8cm -->
   </joint>
 </robot>

Commit message: docs: 更新文档至v1.5，优化激光滤波器配置
主要更新内容：

【激光滤波器配置】
- 调整后方遮挡角度为45°（右侧29° + 左侧16°）
- 采用非对称配置，更精确适应立柱实际遮挡31.2°
- 保留前方315°有效扫描范围

【文档更新】
- 技术文档.md 版本升级至1.5，更新日期2025-12-07
- 快速启动指南.md 添加Foxglove Bridge远程可视化工具
- 连接地址: ws://172.20.10.9:8765

【配置文件更新】
- navigation.rviz: RViz配置优化
- my_robot.urdf.xacro: 机器人URDF模型更新

【新增文件】
- AI_Patrol_Scheme.md: AI巡检方案文档
- robot-arm/: 机械臂相关代码目录
- map4/: 新增地图目录
- test_scripts/TestTool.md: 测试工具文档

【删除文件】
- test_scripts/README.md: 移除旧文档

File: src/robot_bringup_cpp/urdf/my_robot.urdf.xacro (robot description, xacro)
@@ -127,5 +127,5 @@
     <parent link="base_link"/>
     <child link="laser_link"/>
-    <origin xyz="0.258 0 0.318" rpy="0 0 0"/>  <!-- 2025-11-15更新: 底盘高50cm，雷达底部仍离地69.6cm，雷达中心相对base_link为31.8cm -->
+    <origin xyz="0.258 0 0.322" rpy="0 0 0"/>  <!-- 2025-12-07更新: 雷达底部离地70cm，雷达中心离地72cm，相对base_link(39.8cm)为32.2cm -->
   </joint>
 </robot>

Commit message: 🎉 SLAM建图配置优化 - 成功实现回环检测
📋 主要更改：

【SLAM配置优化】slam_toolbox_real.yaml
- minimum_time_interval: 0.15→0.1s (匹配10Hz激光频率)
- minimum_travel_heading: 0.044→0.0175 (1°创建节点，90°旋转90个节点)
- scan_buffer_size: 3000→30000 (支持20分钟建图)
- 回环检测参数放宽(极限宽松模式)：
  · loop_match_minimum_chain_size: 3→1 (单次匹配即可)
  · loop_match_maximum_variance_coarse: 12→30
  · loop_match_minimum_response_coarse: 0.22→0.08
  · loop_match_minimum_response_fine: 0.35→0.15
  · loop_search_maximum_distance: 10→12m
  · loop_search_space_smear_deviation: 0.05→0.1
- angle_variance_penalty: 0.75→1.0 (降低对编码器角度信任)

【激光滤波器】laser_filter.yaml
- 两侧对称遮挡26°(原不对称49°)
- 保留308°有效扫描范围

【里程计协方差】odom_publisher_node.cpp
- yaw协方差: 0.08→0.15 (降低对编码器角度信任)

【快速启动指南】快速启动指南.md
- 新增：建图最佳实践（实测成功方法）
- 新增：速度控制策略（线速度0.01-0.02，角速度0.03-0.1）
- 新增：转角策略（弯角/直角转弯技巧）
- 新增：原地旋转前关键步骤（先探测再转弯）
- 新增：回环检测技巧和成功标志
- 新增：回环偏移变化规律解释
- 新增：实测成功路线图（右下角起点，顺时针）

【新增地图】maps/
- my_map.pgm (368x521像素，2cm分辨率)
- my_map.yaml

🎯 建图成果：
- 回环检测成功：偏差从24.3cm修正到1.5cm
- 角度误差：<1°
- 配置适用于：52°激光盲区 + 编码器旋转误差大的场景

File: src/robot_bringup_cpp/urdf/my_robot.urdf.xacro (robot description, xacro)
@@ -127,5 +127,5 @@
     <parent link="base_link"/>
     <child link="laser_link"/>
-    <origin xyz="0.258 0 0.322" rpy="0 0 0"/>  <!-- 2025-12-07更新: 雷达底部离地70cm，雷达中心离地72cm，相对base_link(39.8cm)为32.2cm -->
+    <origin xyz="0.258 0 0.318" rpy="0 0 0"/>  <!-- 2025-11-15更新: 底盘高50cm，雷达底部仍离地69.6cm，雷达中心相对base_link为31.8cm -->
   </joint>
 </robot>
